File: HVC-CPU-GPM-02/tech.kicad_sch (KiCad schematic)
At the start: 0 parts

Commit message: Rearranged pins on some symbols to simplify schematic wiring Removed schematics for controller PCBs Added PNG version of schematics
Other:
- title: (none) -> Nintendo Famicom Mainboard
Changed lines of the file:
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@@
 	(generator_version "9.0")
 	(paper "A4")
+	(title_block
+		(title "Nintendo Famicom Mainboard")
+		(date "2025-10-30")
+		(rev "1")
+	)
 	(text "31\n32\n33\n34\n35\n36\n37\n38\n39\n40\n41\n42\n43\n44\n45\n46\n47\n48\n49\n50\n51\n52\n53\n54\n55\n56\n57\n58\n59\n60"
 		(exclude_from_sim no)
